File: hardware/New_PCB/usb-c/_autosave-usb-c.sch (KiCad schematic (older format))
At the start: 14 parts, among them J1 USB_C_Receptacle, P1 66200221022, U1 RS6-0505S

Commit message: Gitignore change, and work on DC-DC PCB
Parts:
- P1: symbol USERDEF:66200221022 -> usb-c-rescue:66200221022-USERDEF
- R1: value 10K -> 22K
- U1: symbol USERDEF:RS6-0505S -> usb-c-rescue:RS6-0505S-USERDEF
Other:
- moved on the sheet: C1, C2, C3, D1, D2, D3, J1, L1, L2, P1, R1, R2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
