File: hardware/New_PCB/usb-c/usb-c.sch (KiCad schematic (older format))
At the start: 14 parts, among them J1 USB_C_Receptacle

Commit message: Gitignore change, and work on DC-DC PCB
Parts:
- D3: renamed from D?; footprint (none) -> Diode_SMD:D_0603_1608Metric_Pad1.05x0.95mm_HandSolder
- L1, L2: renamed from L?; value L -> 1µ; footprint (none) -> Inductor_SMD:L_1008_2520Metric
- P1: renamed from P?; symbol USERDEF:66200221022 -> usb-c-rescue:66200221022-USERDEF
- R1: value 10K -> 22K
- U1: renamed from U?; symbol USERDEF:RS6-0505S -> usb-c-rescue:RS6-0505S-USERDEF
- gave numbers to parts that had none: 2
Other:
- moved on the sheet: C1, C2, C3, D1, D2, D3, J1, L1, L2, P1, R1, R2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
